File: pcb.sch (KiCad schematic (older format))
At the start: 30 parts, among them J1 Conn_01x02, J2 Conn_01x03, J3 Conn_01x03, J4 Conn_01x02, J5 Conn_01x02, J6 Conn_02x05_Odd_Even, Q1 2N3904, Q2 2N3904, Q3 2N3904, Q4 2N3904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

Commit message: evan recommmendations
Changed lines of the file:
@@
 PA9
-Wire Wire Line
-	3150 4900 3300 4900
-Connection ~ 3150 4900
-Wire Wire Line
-	3150 4800 3150 4900
-Wire Wire Line
-	3050 4800 3150 4800
-Wire Wire Line
-	3050 4900 3150 4900
 Wire Wire Line
 	3250 7600 3050 7600
@@
 F 3 "" H 7400 1700 50  0001 C CNN
 	1    7400 1700
-	1    0    0    -1
-$EndComp
-$Comp
-L STM32F103C8T6:STM32F103C8T6 U1
-U 1 1 62107107
-P 2050 6300
-F 0 "U1" H 2050 8067 50  0000 C CNN
-F 1 "STM32F103C8T6" H 2050 7976 50  0000 C CNN
-F 2 "STM32F103C8T6:QFP50P900X900X160-48N" H 2050 6300 50  0001 L BNN
-F 3 "" H 2050 6300 50  0001 L BNN
-F 4 "10" H 2050 6300 50  0001 L BNN "PARTREV"
-F 5 "IPC7351B" H 2050 6300 50  0001 L BNN "STANDARD"
-F 6 "ST Microelectronics" H 2050 6300 50  0001 L BNN "MANUFACTURER"
-	1    2050 6300
 	1    0    0    -1
 $EndComp
@@
 Wire Wire Line
 	7350 1050 7350 950
+Wire Wire Line
+	3050 4900 3300 4900
+$Comp
+L STM32F103C8T6:STM32F103C8T6 U1
+U 1 1 62107107
+P 2050 6300
+F 0 "U1" H 2050 8067 50  0000 C CNN
+F 1 "STM32F103C8T6" H 2050 7976 50  0000 C CNN
+F 2 "STM32F103C8T6:QFP50P900X900X160-48N" H 2050 6300 50  0001 L BNN
+F 3 "" H 2050 6300 50  0001 L BNN
+F 4 "10" H 2050 6300 50  0001 L BNN "PARTREV"
+F 5 "IPC7351B" H 2050 6300 50  0001 L BNN "STANDARD"
+F 6 "ST Microelectronics" H 2050 6300 50  0001 L BNN "MANUFACTURER"
+	1    2050 6300
+	1    0    0    -1
+$EndComp
+$Comp
+L power:+3V3 #PWR?
+U 1 1 622124C1
+P 3100 4650
+F 0 "#PWR?" H 3100 4500 50  0001 C CNN
+F 1 "+3V3" H 3115 4823 50  0000 C CNN
+F 2 "" H 3100 4650 50  0001 C CNN
+F 3 "" H 3100 4650 50  0001 C CNN
+	1    3100 4650
+	1    0    0    -1
+$EndComp
+Wire Wire Line
+	3100 4650 3100 4800
+Wire Wire Line
+	3100 4800 3050 4800
 $EndSCHEMATC

Commit message: made changes into pcb, added python code
Parts:
- removed J4, J5: Conn_01x02, Connector_PinHeader_2.54mm:PinHeader_1x02_P2.54mm_Vertical, symbol Connector_Generic:Conn_01x02
- removed J6: Conn_02x05_Odd_Even, Connector_PinHeader_2.54mm:PinHeader_2x05_P2.54mm_Vertical, symbol Connector_Generic:Conn_02x05_Odd_Even
- added C9: 100nF, Capacitor_SMD:C_0603_1608Metric_Pad1.05x0.95mm_HandSolder, symbol device:C
- added J10, J11, J6, J7, J8, J9: Conn_01x03-Connector_Generic, Connector_PinSocket_2.54mm:PinSocket_1x03_P2.54mm_Vertical, symbol pcb-rescue:Conn_01x03-Connector_Generic
- added J4: Conn_01x06, Connector_PinHeader_1.27mm:PinHeader_1x06_P1.27mm_Vertical, symbol Connector_Generic:Conn_01x06
- added R7: 10K, Resistor_SMD:R_1206_3216Metric_Pad1.42x1.75mm_HandSolder, symbol device:R_US
- added SW1: SW_Push, Button_Switch_SMD:SW_SPST_PTS645, symbol Switch:SW_Push
- C1, C2, C3, C4, C5, C6, C7, C8: symbol device:C -> pcb-rescue:C-device
- G1: symbol components_senior_design:GPS_NEO_6M_module -> pcb-rescue:GPS_NEO_6M_module-components_senior_design
- J1: symbol Connector_Generic:Conn_01x02 -> pcb-rescue:Conn_01x02-Connector_Generic
- J2, J3: symbol Connector_Generic:Conn_01x03 -> pcb-rescue:Conn_01x03-Connector_Generic
- Q1, Q2, Q3, Q4: symbol Transistor_BJT:2N3904 -> pcb-rescue:2N3904-Transistor_BJT
- R1, R2, R3, R4, R5, R6: symbol device:R_US -> pcb-rescue:R_US-device
- U1: symbol STM32F103C8T6:STM32F103C8T6 -> pcb-rescue:STM32F103C8T6-STM32F103C8T6
- U2: symbol components_senior_design:Shaft_encoder -> pcb-rescue:Shaft_encoder-components_senior_design
- U3: symbol components_senior_design:compass_accelerometer -> pcb-rescue:compass_accelerometer-components_senior_design
- U4: symbol Regulator_Linear:LM1117-3.3 -> pcb-rescue:LM1117-3.3-Regulator_Linear
- U5: symbol components_senior_design:3v7_to_5V_boost -> pcb-rescue:3v7_to_5V_boost-components_senior_design
Connections:
- net +3V3: now also R7.1
- net +5V: now also J4.1 (Pin_1)
- net GND: now also C9.2, J10.3 (Pin_3), J11.3 (Pin_3), J4.6 (Pin_6), J6.3 (Pin_3), J7.3 (Pin_3), J8.3 (Pin_3), J9.3 (Pin_3), SW1.2
- net NRST: now also C9.1, R7.2, SW1.1
- net PA0: now also J7.1 (Pin_1)
- net PA1: now also J8.1 (Pin_1)
- net PA13: now also J6.1 (Pin_1)
- net PA14: now also J6.2 (Pin_2)
- net PA2: now reaches U1.12 (PA2)
- net PA2: now also J9.1 (Pin_1)
- net PA3: now reaches U1.13 (PA3)
- net PA3: now also J10.1 (Pin_1)
- net PA6: now reaches U1.16 (PA6)
- net PA6: now also J11.1 (Pin_1)
- net RX: now reaches U1.21 (PB10)
- net RX: now also J4.2 (Pin_2)
- net TX: now reaches U1.22 (PB11)
- net TX: now also J4.3 (Pin_3)
- net PB3: no longer names the net of U1.39 (PB3)
- no-connect marks 34 -> 35
Other:
- moved on the sheet: C1, C2, J1, U4, U5

Commit message: final changes to PCB
Parts:
- J4: footprint Connector_PinHeader_1.27mm:PinHeader_1x06_P1.27mm_Vertical -> Connector_Hirose:Hirose_DF13-06P-1.25DSA_1x06_P1.25mm_Vertical
- R1, R2, R3, R4, R5, R6, R7: footprint Resistor_SMD:R_1206_3216Metric_Pad1.42x1.75mm_HandSolder -> Resistor_SMD:R_0805_2012Metric_Pad1.15x1.40mm_HandSolder
Changed lines of the file:
@@
 F 0 "R1" V 1395 1800 50  0000 C CNN
 F 1 "4.7K" V 1486 1800 50  0000 C CNN
-F 2 "Resistor_SMD:R_1206_3216Metric_Pad1.42x1.75mm_HandSolder" V 1640 1790 50  0001 C CNN
+F 2 "Resistor_SMD:R_0805_2012Metric_Pad1.15x1.40mm_HandSolder" V 1640 1790 50  0001 C CNN
 F 3 "~" H 1600 1800 50  0001 C CNN
 	1    1600 1800
@@
 F 0 "R2" H 2368 1396 50  0000 L CNN
 F 1 "4.7K" H 2368 1305 50  0000 L CNN
-F 2 "Resistor_SMD:R_1206_3216Metric_Pad1.42x1.75mm_HandSolder" V 2340 1340 50  0001 C CNN
+F 2 "Resistor_SMD:R_0805_2012Metric_Pad1.15x1.40mm_HandSolder" V 2340 1340 50  0001 C CNN
 F 3 "~" H 2300 1350 50  0001 C CNN
 	1    2300 1350
@@
 F 0 "R3" H 3568 1396 50  0000 L CNN
 F 1 "1K" H 3568 1305 50  0000 L CNN
-F 2 "Resistor_SMD:R_1206_3216Metric_Pad1.42x1.75mm_HandSolder" V 3540 1340 50  0001 C CNN
+F 2 "Resistor_SMD:R_0805_2012Metric_Pad1.15x1.40mm_HandSolder" V 3540 1340 50  0001 C CNN
 F 3 "~" H 3500 1350 50  0001 C CNN
 	1    3500 1350
@@
 F 0 "R6" H 3618 3096 50  0000 L CNN
 F 1 "1K" H 3618 3005 50  0000 L CNN
-F 2 "Resistor_SMD:R_1206_3216Metric_Pad1.42x1.75mm_HandSolder" V 3590 3040 50  0001 C CNN
+F 2 "Resistor_SMD:R_0805_2012Metric_Pad1.15x1.40mm_HandSolder" V 3590 3040 50  0001 C CNN
 F 3 "~" H 3550 3050 50  0001 C CNN
 	1    3550 3050
@@
 F 0 "R5" H 2418 3096 50  0000 L CNN
 F 1 "4.7K" H 2418 3005 50  0000 L CNN
-F 2 "Resistor_SMD:R_1206_3216Metric_Pad1.42x1.75mm_HandSolder" V 2390 3040 50  0001 C CNN
+F 2 "Resistor_SMD:R_0805_2012Metric_Pad1.15x1.40mm_HandSolder" V 2390 3040 50  0001 C CNN
 F 3 "~" H 2350 3050 50  0001 C CNN
 	1    2350 3050
@@
 F 0 "R4" V 1445 3500 50  0000 C CNN
 F 1 "4.7K" V 1536 3500 50  0000 C CNN
-F 2 "Resistor_SMD:R_1206_3216Metric_Pad1.42x1.75mm_HandSolder" V 1690 3490 50  0001 C CNN
+F 2 "Resistor_SMD:R_0805_2012Metric_Pad1.15x1.40mm_HandSolder" V 1690 3490 50  0001 C CNN
 F 3 "~" H 1650 3500 50  0001 C CNN
 	1    1650 3500
@@
 F 0 "R7" H 4068 6646 50  0000 L CNN
 F 1 "10K" H 4068 6555 50  0000 L CNN
-F 2 "Resistor_SMD:R_1206_3216Metric_Pad1.42x1.75mm_HandSolder" V 4040 6590 50  0001 C CNN
+F 2 "Resistor_SMD:R_0805_2012Metric_Pad1.15x1.40mm_HandSolder" V 4040 6590 50  0001 C CNN
 F 3 "~" H 4000 6600 50  0001 C CNN
 	1    4000 6600
@@
 F 0 "J4" H 9030 5592 50  0000 L CNN
 F 1 "Conn_01x06" H 9030 5501 50  0000 L CNN
-F 2 "Connector_PinHeader_1.27mm:PinHeader_1x06_P1.27mm_Vertical" H 8950 5600 50  0001 C CNN
+F 2 "Connector_Hirose:Hirose_DF13-06P-1.25DSA_1x06_P1.25mm_Vertical" H 8950 5600 50  0001 C CNN
 F 3 "~" H 8950 5600 50  0001 C CNN
 	1    8950 5600

Commit message: second round pcb
Parts:
- added J12: USB_B_Micro, Connector_USB:USB_Micro-B_Molex-105133-0031, symbol Connector:USB_B_Micro
- added J5: Conn_02x03, Connector_PinHeader_2.54mm:PinHeader_2x03_P2.54mm_Vertical, symbol Connector_Generic:Conn_02x03_Odd_Even
- added R10, R11: 20R, Resistor_SMD:R_0805_2012Metric_Pad1.15x1.40mm_HandSolder, symbol device:R_US
- added R12: 4.7K, Resistor_SMD:R_0805_2012Metric_Pad1.15x1.40mm_HandSolder, symbol device:R_US
- added R8, R9: 100K, Resistor_SMD:R_0805_2012Metric_Pad1.15x1.40mm_HandSolder, symbol pcb-rescue:R_US-device
- J6: footprint Connector_PinSocket_2.54mm:PinSocket_1x03_P2.54mm_Vertical -> Connector_PinHeader_2.54mm:PinHeader_1x03_P2.54mm_Horizontal
Connections:
- net +3V3: now also J5.1 (Pin_1), J5.2 (Pin_2)
- net +5V: now also J12.1 (VBUS), R12.2
- net GND: now also J12.4 (ID), J12.5 (GND), J12.6 (Shield), J5.5 (Pin_5), J5.6 (Pin_6); no longer U1.44 (BOOT0)
- net BOOT1: now reaches U1.20 (PB2)
- net BOOT1: now also R9.2
- net PA11: now reaches U1.32 (PA11)
- net PA11: now also R11.2
- net PA12: now reaches U1.33 (PA12)
- net PA12: now also R10.2, R12.1
- new net: J12.2 (D-), R11.1
- new net: J12.3 (D+), R10.1
- new net: J5.3 (Pin_3), R8.2
- new net: J5.4 (Pin_4), R9.1
- new net BOOT0: R8.1, U1.44 (BOOT0)
- no-connect marks 35 -> 32
Other:
- moved on the sheet: C9, J6, R7, SW1
